Commit message: Update README and MoveIt instructions

File: src/my_so101_robot_description_package/urdf/my_so101_robot.urdf.xacro (robot description, xacro)
@@ -7,10 +7,11 @@
   <xacro:arg name="sim_gazebo_classic" default="false"/>
   <xacro:arg name="use_mock_hardware" default="false"/>
-  <xacro:arg name="mock_sensor_commands" default="false"/>
+  <xacro:arg name="mock_sensor_commands" default="true"/>
   <xacro:arg name="initial_positions_file" default="$(find so101_robot_description)/urdf/initial_positions.yaml"/>
-  <xacro:arg name="controller_config_file" default="$(find so101_robot_bringup)/config/controllers.yaml"/>
+  <xacro:arg name="controller_config_file" default="$(find so101_robot_bringup)/config/sub_controllers.yaml"/>
   <xacro:arg name="usb_port" default="/dev/ttyACM0"/>
   <xacro:arg name="recalibrate" default="false"/>
   <xacro:arg name="arm" default="follower"/>
+  <xacro:arg name="namespace" default=""/>
   <xacro:arg name="role" default="follower"/>
   <xacro:include filename="$(find so101_robot_description)/urdf/my_so101_robot/my_so101_robot_macro.xacro" />
@@ -33,4 +34,5 @@
     recalibrate="$(arg recalibrate)"
     arm="$(arg arm)"
+    namespace="$(arg namespace)"
     role="$(arg role)"
   />

File: src/my_so101_robot_description_package/urdf/my_so101_robot/my_so101_robot_macro.ros2_control.xacro (robot description, xacro)
@@ -3,5 +3,5 @@
     <xacro:macro name="so101_ros2_control" params="
                  name:=so101
-                 prefix
+                 prefix:=''
                  use_sim:=false
                  sim_gazebo:=false
@@ -14,4 +14,5 @@
                  recalibrate:=false
                  arm:=follower
+                 namespace:=''
                  role:=follower
                  ">
@@ -24,5 +25,5 @@
                     name="gazebo_ros2_control">
                     <ros>
-                        <namespace>/${arm}</namespace>
+                        <namespace>/${namespace}</namespace>
                     </ros>
                     <parameters>${controller_config_file}</parameters>
@@ -37,5 +38,5 @@
                     name="gz_ros2_control::GazeboSimROS2ControlPlugin">
                     <ros>
-                        <namespace>/${arm}</namespace>
+                        <namespace>/${namespace}</namespace>
                     </ros>
                     <parameters>${controller_config_file}</parameters>

File: src/my_so101_robot_description_package/urdf/so101_moveit_entry.urdf (robot description, URDF)
Before this commit: robot so101, 10 links, 9 joints
Joints:
- joint joint1: limit lower=-1.91986 upper=1.91986 effort=10.0 velocity=10.0 -> lower=-1.91986 upper=1.91986 effort=10 velocity=10
- joint joint2: limit lower=-1.74533 upper=1.74533 effort=10.0 velocity=10.0 -> lower=-1.74533 upper=1.74533 effort=10 velocity=10
- joint joint3: limit lower=-1.74533 upper=1.5708 effort=10.0 velocity=10.0 -> lower=-1.74533 upper=1.5708 effort=10 velocity=10
- joint joint4: limit lower=-1.65806 upper=1.65806 effort=10.0 velocity=10.0 -> lower=-1.65806 upper=1.65806 effort=10 velocity=10
- joint joint5: limit lower=-2.74385 upper=2.84121 effort=10.0 velocity=10.0 -> lower=-2.74385 upper=2.84121 effort=10 velocity=10
- joint joint6: limit lower=-0.174533 upper=1.74533 effort=10.0 velocity=10.0 -> lower=-0.174533 upper=1.74533 effort=10 velocity=10

File: src/my_so101_robot_moveit_package/config/so101.urdf.xacro (robot description, xacro)
@@ -1,9 +1,10 @@
 <?xml version="1.0"?>
 <robot xmlns:xacro="http://www.ros.org/wiki/xacro" name="so101">
-    <xacro:arg name="initial_positions_file" default="initial_positions.yaml" />
+    <!-- <xacro:arg name="initial_positions_file" default="initial_positions.yaml" /> -->
     <!-- Import so101 urdf file -->
     <xacro:include filename="$(find so101_robot_description)/urdf/my_so101_robot.urdf.xacro" />
+    <!-- <xacro:include filename="$(find so101_robot_description)/urdf/so101_moveit_entry.urdf" /> -->
     <!-- Import control_xacro -->
-    <xacro:include filename="so101.ros2_control.xacro" />
-    <xacro:so101_ros2_control name="FakeSystem" initial_positions_file="$(arg initial_positions_file)"/>
+    <!-- <xacro:include filename="so101.ros2_control.xacro" /> -->
+    <!-- <xacro:so101_ros2_control name="FakeSystem" initial_positions_file="$(arg initial_positions_file)"/> -->
 </robot>

Commit message: Finalisation Teleop Launch

File: src/my_so101_robot_description_package/urdf/my_so101_robot.urdf.xacro (robot description, xacro)
@@ -15,10 +15,19 @@
   <xacro:arg name="namespace" default=""/>
   <xacro:arg name="role" default="follower"/>
+  <xacro:arg name="include_world" default="true"/>
   <xacro:include filename="$(find so101_robot_description)/urdf/my_so101_robot/my_so101_robot_macro.xacro" />
   <xacro:include filename="$(find so101_robot_description)/urdf/my_so101_robot/my_so101_robot_macro.ros2_control.xacro" />
-  <link name="world"/>
-  <xacro:so101 prefix="$(arg prefix)" parent="world">
-    <origin xyz="0 0 0" rpy="0 0 0"/> <!-- position robot in the world -->
+  <xacro:so101
+    prefix="$(arg prefix)">
   </xacro:so101>
+  <xacro:if value="$(arg include_world)">
+    <link name="world"/>
+    <!-- Joint from environment to base -->
+    <joint name="$(arg prefix)base_joint" type="fixed">
+      <origin xyz="0 0 0" rpy="0 0 0"/> <!-- position robot in the world -->
+      <parent link="world"/>
+      <child link="$(arg prefix)base"/>
+    </joint>
+  </xacro:if>
   <xacro:so101_ros2_control
     name="$(arg name)"

File: src/my_so101_robot_description_package/urdf/my_so101_robot/my_so101_robot_macro.xacro (robot description, xacro)
@@ -1,5 +1,5 @@
 <?xml version="1.0" encoding="UTF-8"?>
 <robot xmlns:xacro="http://wiki.ros.org/xacro">
-  <xacro:macro name="so101" params="prefix parent *origin">
+  <xacro:macro name="so101" params="prefix">
     <!-- LINKS -->
     <!-- base link -->
@@ -410,10 +410,4 @@
       <limit effort="10" velocity="10" lower="-1.91986" upper="1.91986"/>
     </joint>
-    <!-- Joint from environment to base -->
-    <joint name="${prefix}base_joint" type="fixed">
-      <xacro:insert_block name="origin"/>
-      <parent link="${parent}"/>
-      <child link="${prefix}base"/>
-    </joint>
   </xacro:macro>
 </robot>
